File: hardware/v2.0/bz-hat/bz-hat.sch (KiCad schematic (older format))
At the start: 48 parts, among them J1 LineIN, J2 LineOUT, J3 Headphones, J4 Raspberry_Pi_4, J5 CVs+CLK_connector, J6 NHD-2.23-12832UCB3, SW1 BTN_f, SW2 BTN_big, SW3 BTN_1, SW4 BTN_2, SW5 BTN_3, U1 MCP3004, U2 WM8731, U3 MCP3004

Commit message: logo + gerbers + JLPCB refs. to symbols
Parts:
- C1, C2: LCSC (none) -> C1603
- C10, C11, C15, C19, C9: LCSC (none) -> C7171
- C12, C14, C16, C17: LCSC (none) -> C14663
- C13: LCSC (none) -> C24497
- C18, C20, C3, C4, C7, C8: LCSC (none) -> C7176
- C5, C6: LCSC (none) -> C127327
- R1, R2, R5, R6: LCSC (none) -> C4382
- R10, R7, R8, R9: LCSC (none) -> C17713
- R3, R4: LCSC (none) -> C17408
- U1, U3: LCSC (none) -> C512186
- U2: LCSC (none) -> C323837
Changed lines of the file:
@@
 F 2 "custom:SSOP28-0.65-10.2X5.2MM" H 6750 3650 50  0001 C CNN
 F 3 "" H 6750 3650 50  0001 C CNN
+F 4 " C323837" H 6750 2800 50  0001 C CNN "LCSC"
 	1    6750 2800
 	1    0    0    -1
@@
 F 2 "Resistor_SMD:R_0805_2012Metric" V 2380 5100 50  0001 C CNN
 F 3 "~" H 2450 5100 50  0001 C CNN
+F 4 "C4382" V 2450 5100 50  0001 C CNN "LCSC"
 	1    2450 5100
 	0    -1   1    0
@@
 F 2 "Resistor_SMD:R_0805_2012Metric" V 2630 5300 50  0001 C CNN
 F 3 "~" H 2700 5300 50  0001 C CNN
+F 4 "C4382" V 2700 5300 50  0001 C CNN "LCSC"
 	1    2700 5300
 	1    0    0    1
@@
 F 2 "Capacitor_SMD:C_0603_1608Metric" H 3138 5150 50  0001 C CNN
 F 3 "~" H 3100 5300 50  0001 C CNN
+F 4 "C1603" H 3100 5300 50  0001 C CNN "LCSC"
 	1    3100 5300
 	-1   0    0    -1
@@
 F 2 "Capacitor_Tantalum_SMD:CP_EIA-3216-18_Kemet-A" H 3438 4950 50  0001 C CNN
 F 3 "~" H 3400 5100 50  0001 C CNN
+F 4 "C7176" V 3400 5100 50  0001 C CNN "LCSC"
 	1    3400 5100
 	0    1    -1   0
@@
 F 2 "Resistor_SMD:R_0805_2012Metric" V 2380 5950 50  0001 C CNN
 F 3 "~" H 2450 5950 50  0001 C CNN
+F 4 "C4382" V 2450 5950 50  0001 C CNN "LCSC"
 	1    2450 5950
 	0    -1   1    0
@@
 F 2 "Resistor_SMD:R_0805_2012Metric" V 2630 6150 50  0001 C CNN
 F 3 "~" H 2700 6150 50  0001 C CNN
+F 4 "C4382" V 2700 6150 50  0001 C CNN "LCSC"
 	1    2700 6150
 	1    0    0    1
@@
 F 2 "Capacitor_SMD:C_0603_1608Metric" H 3138 6000 50  0001 C CNN
 F 3 "~" H 3100 6150 50  0001 C CNN
+F 4 "C1603" H 3100 6150 50  0001 C CNN "LCSC"
 	1    3100 6150
 	-1   0    0    -1
@@
 F 2 "Capacitor_Tantalum_SMD:CP_EIA-3216-18_Kemet-A" H 3438 5800 50  0001 C CNN
 F 3 "~" H 3400 5950 50  0001 C CNN
+F 4 "C7176" V 3400 5950 50  0001 C CNN "LCSC"
 	1    3400 5950
 	0    1    -1   0
@@
 F 2 "Capacitor_Tantalum_SMD:CP_EIA-3216-18_Kemet-A" H 3388 1650 50  0001 C CNN
 F 3 "~" H 3350 1800 50  0001 C CNN
+F 4 "C7176" V 3350 1800 50  0001 C CNN "LCSC"
 	1    3350 1800
 	0    1    1    0
@@
 F 2 "Resistor_SMD:R_0805_2012Metric" V 2880 1950 50  0001 C CNN
 F 3 "~" H 2950 1950 50  0001 C CNN
+F 4 " C17713" H 2950 1950 50  0001 C CNN "LCSC"
 	1    2950 1950
 	1    0    0    -1
@@
 F 2 "Resistor_SMD:R_0805_2012Metric" V 2430 1800 50  0001 C CNN
 F 3 "~" H 2500 1800 50  0001 C CNN
+F 4 "C17408" V 2500 1800 50  0001 C CNN "LCSC"
 	1    2500 1800
 	0    1    1    0
@@
 F 2 "Capacitor_Tantalum_SMD:CP_EIA-3216-18_Kemet-A" H 3438 2450 50  0001 C CNN
 F 3 "~" H 3400 2600 50  0001 C CNN
+F 4 "C7176" V 3400 2600 50  0001 C CNN "LCSC"
 	1    3400 2600
 	0    1    1    0
@@
 F 2 "Resistor_SMD:R_0805_2012Metric" V 2930 2750 50  0001 C CNN
 F 3 "~" H 3000 2750 50  0001 C CNN
+F 4 " C17713" H 3000 2750 50  0001 C CNN "LCSC"
 	1    3000 2750
 	1    0    0    -1
@@
 F 2 "Resistor_SMD:R_0805_2012Metric" V 2480 2600 50  0001 C CNN
 F 3 "~" H 2550 2600 50  0001 C CNN
+F 4 "C17408" V 2550 2600 50  0001 C CNN "LCSC"
 	1    2550 2600
 	0    1    1    0
@@
 F 2 "Capacitor_SMD:CP_Elec_6.3x7.7" H 3438 3300 50  0001 C CNN
 F 3 "~" H 3400 3450 50  0001 C CNN
+F 4 " C127327" V 3400 3450 50  0001 C CNN "LCSC"
 	1    3400 3450
 	0    1    1    0
@@
 F 2 "Resistor_SMD:R_0805_2012Metric" V 2930 4400 50  0001 C CNN
 F 3 "~" H 3000 4400 50  0001 C CNN
+F 4 " C17713" H 3000 4400 50  0001 C CNN "LCSC"
 	1    3000 4400
 	1    0    0    -1
@@
 F 2 "Capacitor_SMD:CP_Elec_6.3x7.7" H 3438 4100 50  0001 C CNN
 F 3 "~" H 3400 4250 50  0001 C CNN
+F 4 " C127327" V 3400 4250 50  0001 C CNN "LCSC"
 	1    3400 4250
 	0    1    1    0
@@
 F 2 "Resistor_SMD:R_0805_2012Metric" V 2930 3600 50  0001 C CNN
 F 3 "~" H 3000 3600 50  0001 C CNN
+F 4 " C17713" H 3000 3600 50  0001 C CNN "LCSC"
 	1    3000 3600
 	1    0    0    -1
@@
 F 2 "Capacitor_Tantalum_SMD:CP_EIA-3216-18_Kemet-A" H 7638 1950 50  0001 C CNN
 F 3 "~" H 7600 2100 50  0001 C CNN
+F 4 " C7171" H 7600 2100 50  0001 C CNN "LCSC"
 	1    7600 2100
 	-1   0    0    1
@@
 F 2 "Capacitor_SMD:C_0603_1608Metric" H 8038 1950 50  0001 C CNN
 F 3 "~" H 8000 2100 50  0001 C CNN
+F 4 "C14663" H 8000 2100 50  0001 C CNN "LCSC"
 	1    8000 2100
 	-1   0    0    -1
@@
 F 2 "Capacitor_SMD:C_0603_1608Metric" H 8138 3350 50  0001 C CNN
 F 3 "~" H 8100 3500 50  0001 C CNN
+F 4 " C7171" H 8100 3500 50  0001 C CNN "LCSC"
 	1    8100 3500
 	1    0    0    -1
@@
 F 2 "Capacitor_SMD:C_0603_1608Metric" H 7738 3350 50  0001 C CNN
 F 3 "~" H 7700 3500 50  0001 C CNN
+F 4 "C14663" H 7700 3500 50  0001 C CNN "LCSC"
 	1    7700 3500
 	1    0    0    1
@@
 F 2 "Capacitor_Tantalum_SMD:CP_EIA-3216-18_Kemet-A" H 5188 1850 50  0001 C CNN
 F 3 "~" H 5150 2000 50  0001 C CNN
+F 4 " C7171" H 5150 2000 50  0001 C CNN "LCSC"
 	1    5150 2000
 	1    0    0    1
@@
 F 2 "Capacitor_SMD:C_0603_1608Metric" H 5588 1850 50  0001 C CNN
 F 3 "~" H 5550 2000 50  0001 C CNN
+F 4 "C14663" H 5550 2000 50  0001 C CNN "LCSC"
 	1    5550 2000
 	-1   0    0    1
@@
 F 2 "Capacitor_Tantalum_SMD:CP_EIA-3216-18_Kemet-A" H 5188 2850 50  0001 C CNN
 F 3 "~" H 5150 3000 50  0001 C CNN
+F 4 " C7171" H 5150 3000 50  0001 C CNN "LCSC"
 	1    5150 3000
 	1    0    0    -1
@@
 F 2 "Capacitor_SMD:C_1206_3216Metric" H 5588 2850 50  0001 C CNN
 F 3 "~" H 5550 3000 50  0001 C CNN
+F 4 "C24497" H 5550 3000 50  0001 C CNN "LCSC"
 	1    5550 3000
 	-1   0    0    -1
@@
 F 2 "Capacitor_Tantalum_SMD:CP_EIA-3216-18_Kemet-A" H 5188 3450 50  0001 C CNN
 F 3 "~" H 5150 3600 50  0001 C CNN
+F 4 " C7171" H 5150 3600 50  0001 C CNN "LCSC"
 	1    5150 3600
 	1    0    0    -1
@@
 F 2 "Capacitor_SMD:C_0603_1608Metric" H 5588 3450 50  0001 C CNN
 F 3 "~" H 5550 3600 50  0001 C CNN
+F 4 "C14663" H 5550 3600 50  0001 C CNN "LCSC"
 	1    5550 3600
 	-1   0    0    -1
@@
 F 2 "Package_SO:SOIC-14_3.9x8.7mm_P1.27mm" H 7550 4950 50  0001 C CNN
 F 3 "http://ww1.microchip.com/downloads/en/DeviceDoc/21295C.pdf" H 7550 4950 50  0001 C CNN
+F 4 " C512186" H 6650 5250 50  0001 C CNN "LCSC"
 	1    6650 5250
 	1    0    0    -1
@@
 F 2 "Package_SO:SOIC-14_3.9x8.7mm_P1.27mm" H 14250 1900 50  0001 C CNN
 F 3 "http://ww1.microchip.com/downloads/en/DeviceDoc/21295C.pdf" H 14250 1900 50  0001 C CNN
+F 4 " C512186" H 13350 2200 50  0001 C CNN "LCSC"
 	1    13350 2200
 	1    0    0    -1
@@
 F 2 "Capacitor_Tantalum_SMD:CP_EIA-3216-18_Kemet-A" H 8038 5150 50  0001 C CNN
 F 3 "~" H 8000 5300 50  0001 C CNN
+F 4 " C7176" H 8000 5300 50  0001 C CNN "LCSC"
 	1    8000 5300
 	1    0    0    -1
@@
 F 2 "Capacitor_Tantalum_SMD:CP_EIA-3216-18_Kemet-A" H 14738 2050 50  0001 C CNN
 F 3 "~" H 14700 2200 50  0001 C CNN
+F 4 " C7176" H 14700 2200 50  0001 C CNN "LCSC"
 	1    14700 2200
 	1    0    0    -1
