File: hardware/v2.0/bz-hat/bz-hat.sch (KiCad schematic (older format))
At the start: 48 parts, among them J1 LineIN, J2 LineOUT, J3 Headphones, J4 Raspberry_Pi_4, J5 CVs+CLK_connector, J6 NHD-2.23-12832UCB3, SW1 BTN_f, SW2 BTN_big, SW3 BTN_1, SW4 BTN_2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

Commit message: Fixed C19 wrong footprint
Parts:
- C19: footprint Capacitor_SMD:C_0603_1608Metric -> Capacitor_Tantalum_SMD:CP_EIA-3216-18_Kemet-A
Changed lines of the file:
@@
 F 0 "C19" H 7982 3454 50  0000 R CNN
 F 1 "10uF" H 7982 3545 50  0000 R CNN
-F 2 "Capacitor_SMD:C_0603_1608Metric" H 8138 3350 50  0001 C CNN
+F 2 "Capacitor_Tantalum_SMD:CP_EIA-3216-18_Kemet-A" H 8138 3350 50  0001 C CNN
 F 3 "~" H 8100 3500 50  0001 C CNN
 F 4 " C7171" H 8100 3500 50  0001 C CNN "LCSC"

Commit message: Added interactive BOM with manufacturer, distributor, price fields
Parts:
- C1, C2: Distributor (none) -> JLCPCB parts; Manufacturer name (none) -> Samsung Electro-Mechanics; Manufacturer part # (none) -> CL10B221KB8NNNC; Price (€) (none) -> 0.006
- C10, C11, C15, C19, C9: Distributor (none) -> JLCPCB parts; LCSC C7171 -> C7171; Manufacturer name (none) -> AVX; Manufacturer part # (none) -> TAJA106K016RNJ; Price (€) (none) -> 0.17
- C12, C14, C16, C17: Distributor (none) -> JLCPCB parts; Manufacturer name (none) -> Yageo; Manufacturer part # (none) -> CC0603KRX7R9BB104; Price (€) (none) -> 0.006
- C13: Distributor (none) -> JLCPCB parts; Manufacturer name (none) -> Samsung Electro-Mechanics; Manufacturer part # (none) -> CL31B104KBCNNNC; Price (€) (none) -> 0.02
- C18, C20: Distributor (none) -> JLCPCB parts; LCSC C7176 -> C7176; Manufacturer name (none) -> AVX; Manufacturer part # (none) -> TAJA105K035RNJ; Price (€) (none) -> 0.13
- C3, C4, C7, C8: Distributor (none) -> JLCPCB parts; Manufacturer name (none) -> AVX; Manufacturer part # (none) -> TAJA105K035RNJ; Price (€) (none) -> 0.13
- C5, C6: Distributor (none) -> JLCPCB parts; LCSC C127327 -> C127327; Manufacturer name (none) -> LELON; Manufacturer part # (none) -> VES221M1CTR-0607; Price (€) (none) -> 0.04
- J1, J2, J3: Distributor (none) -> https://eu.mouser.com/ProductDetail/CUI-Devices/SJ1-3533NG/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; LCSC (none) -> -; Manufacturer name (none) -> CUI Devices; Manufacturer part # (none) -> SJ1-3533NG; Price (€) (none) -> 0.98
- J4: Distributor (none) -> https://eu.mouser.com/ProductDetail/Adafruit/1992/?qs=GURaw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; LCSC (none) -> -; Manufacturer name (none) -> Adafruit; Price (€) (none) -> 2.50
- J5: Distributor (none) -> https://eu.mouser.com/ProductDetail/Preci-dip/801-87-004-10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; LCSC (none) -> -; Manufacturer name (none) -> Preci-dip; Manufacturer part # (none) -> 801-87-004-10-001101; Price (€) (none) -> 0.36
- J6: Distributor (none) -> https://eu.mouser.com/ProductDetail/Newhaven-Display/NHD-22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; LCSC (none) -> -; Manufacturer name (none) -> Newhaven Displays; Manufacturer part # (none) -> NHD-2.23-12832UCB3; Price (€) (none) -> 23.43
- R1, R2, R5, R6: Distributor (none) -> JLCPCB parts; Manufacturer name (none) -> Uniroyal Elec; Manufacturer part # (none) -> 0805W8F5601T5E; Price (€) (none) -> 0.004
- R10, R7, R8, R9: Distributor (none) -> JLCPCB parts; LCSC C17713 -> C17713; Manufacturer name (none) -> Uniroyal Elec; Manufacturer part # (none) -> 0805W8F4702T5E; Price (€) (none) -> 0.004
- R3, R4: Distributor (none) -> JLCPCB parts; Manufacturer name (none) -> Uniroyal Elec; Manufacturer part # (none) -> 0805W8F1000T5E; Price (€) (none) -> 0.003
- RV1, RV2, RV3, RV4: Distributor (none) -> https://eu.mouser.com/ProductDetail/Alps-Alpine/RK09L114001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; LCSC (none) -> -; Manufacturer name (none) -> Alps; Manufacturer part # (none) -> RK09L114001T; Price (€) (none) -> 1.5
- SW1, SW3, SW4, SW5: Distributor (none) -> https://eu.mouser.com/ProductDetail/E-Switch/TL1100F160Q6JB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; LCSC (none) -> -; Manufacturer name (none) -> E-Switch; Manufacturer part # (none) -> TL1100F160Q6JBLK; Price (€) (none) -> 0.65
- SW2: Distributor (none) -> https://eu.mouser.com/ProductDetail/E-Switch/PB300STQ/?qs=4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; LCSC (none) -> -; Manufacturer name (none) -> E-Switch; Manufacturer part # (none) -> PB300STQ; Price (€) (none) -> 1.41
- U1, U3: Distributor (none) -> https://www.mouser.it/ProductDetail/Microchip-Technology/MC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; LCSC C512186 -> -; Manufacturer name (none) -> Microchip Technology; Manufacturer part # (none) -> MCP3004-I/SL; Price (€) (none) -> 1.85
- U2: Distributor (none) -> https://www.mouser.it/ProductDetail/Cirrus-Logic/WM8731SEDS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; LCSC C323837 -> -; Manufacturer name (none) -> Cirrus Logic; Manufacturer part # (none) -> WM8731SEDS/V; Price (€) (none) -> 3.62

Commit message: symbols update and rm jupyter checkpoints
Parts:
- J1, J2, J3: symbol custom:AudioJack3_numbered -> bz-hat-rescue:AudioJack3_numbered-custom
- J4: symbol Connector:Raspberry_Pi_4 -> bz-hat-rescue:Raspberry_Pi_4-Connector
- U1, U3: symbol Analog_ADC:MCP3004 -> bz-hat-rescue:MCP3004-Analog_ADC
- U2: symbol custom:WM8731 -> bz-hat-rescue:WM8731-custom
Changed lines of the file:
@@
 $EndDescr
 $Comp
-L custom:WM8731 U2
+L bz-hat-rescue:WM8731-custom U2
 U 1 1 5E566C4B
 P 6750 2800
@@
 	5900 2750 6200 2750
 $Comp
-L custom:AudioJack3_numbered J1
+L bz-hat-rescue:AudioJack3_numbered-custom J1
 U 1 1 5E660B0F
 P 1550 5550
@@
 $EndComp
 $Comp
-L custom:AudioJack3_numbered J2
+L bz-hat-rescue:AudioJack3_numbered-custom J2
 U 1 1 5E66FF01
 P 1750 2300
@@
 Connection ~ 3000 3450
 $Comp
-L custom:AudioJack3_numbered J3
+L bz-hat-rescue:AudioJack3_numbered-custom J3
 U 1 1 5E67CC5E
 P 1800 3850
@@
 	7300 2650 7600 2650
 $Comp
-L Analog_ADC:MCP3004 U1
+L bz-hat-rescue:MCP3004-Analog_ADC U1
 U 1 1 6034A0E0
 P 6650 5250
@@
 $EndComp
 $Comp
-L Analog_ADC:MCP3004 U3
+L bz-hat-rescue:MCP3004-Analog_ADC U3
 U 1 1 6034D84F
 P 13350 2200
@@
 	2950 10250 3000 10250
 $Comp
-L Connector:Raspberry_Pi_4 J4
+L bz-hat-rescue:Raspberry_Pi_4-Connector J4
 U 1 1 60411F78
 P 2800 8950
